File: Breakout/Breakout.brd (EAGLE design)
At the start: 60.6 x 48.2 mm, 6 parts, among them J1 POWER_JACKSMD

Commit message: Updated stencil text Added PCA9685 and ITG3200 shields
Other:
- board text added: "Nerduino Breakout Shield www.nerduino.com"
- board text removed: "Nerduino Breakout Shield"
Changed lines of the file:
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@@
 <wire x1="70.79" y1="64.76" x2="10.16" y2="64.76" width="0" layer="20"/>
 <wire x1="10.16" y1="64.76" x2="10.16" y2="16.51" width="0" layer="20"/>
-<text x="21.59" y="36.83" size="1.778" layer="1">Nerduino
-Breakout Shield</text>
+<text x="21.59" y="36.83" size="1.778" layer="121">Nerduino
+Breakout Shield
+www.nerduino.com</text>
 </plain>
 <attributes>

Commit message: Added OLED Shield Added LiPo Battery Charger Shield Updated outlines of all shields to match the cutout of the nodemcu board
Parts:
- moved J1 5.14 mm to (63.8, 39.9)
- moved U$1 5.09 mm to (34.3, 34.0)
Connections:
- removed net N$22: J1.VIN0, U$1.14, X3.5
- new net GND: J1.VIN0, U$1.10, U$1.14, U$1.17, U$1.24, X3.5
- new net N$26: U$1.13, X3.3
Routing:
- net N$22: track 60.0 -> 0.00 mm
- net GND: track 0.00 -> 31.7 mm
- net N$26: track 0.00 -> 11.3 mm
- net N$21: track 30.4 -> 39.1 mm
- net N$6: track 16.3 -> 10.6 mm
- net N$2: track 25.4 -> 20.1 mm
- net N$3: track 23.0 -> 18.0 mm
- net N$1: track 24.5 -> 19.6 mm
- net N$5: track 18.0 -> 13.2 mm
- net N$8: track 15.2 -> 10.5 mm
- net N$19: track 17.5 -> 13.0 mm
- net N$23: track 26.1 -> 21.7 mm
- net N$18: track 14.6 -> 10.4 mm
- net N$4: track 19.7 -> 15.6 mm
- net N$9: track 13.5 -> 9.47 mm
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- added copper zone on layer 16, net GND
- removed copper zone on layer 1, net N$24
Other:
- board size 60.6 x 48.2 mm -> 62.2 x 47.7 mm
- board text added: "NERDUINO Breakout Shield www.nerduino.com"
- board text removed: "Nerduino Breakout Shield www.nerduino.com"

Commit message: Updated the i2c pins to all shields to use d11/d12  as these pins will have dual use with the upcoming wifimcu Added FM24W256  Fram shield Added X95840 Digital potentiometer Shield Added AD5696 DAC Shield
Connections:
- net GND: no longer U$1.24
Changed lines of the file:
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@@
 <contactref element="U$1" pad="10"/>
 <contactref element="U$1" pad="14"/>
-<contactref element="U$1" pad="24"/>
 <contactref element="U$1" pad="17"/>
 <wire x1="63.754" y1="45.578" x2="69.992" y2="45.578" width="0.6096" layer="1"/>
