File: Breakout/Breakout.sch (EAGLE design)
At the start: 6 parts, among them J1 POWER_JACKSMD

Commit message: Added OLED Shield Added LiPo Battery Charger Shield Updated outlines of all shields to match the cutout of the nodemcu board
Connections:
- removed net N$22: J1.PWR, U$1.GND$14, X3-5.KL
- new net GND: J1.PWR, U$1.GND$10, U$1.GND$14, U$1.GND$17, U$1.GND$24, X3-5.KL
- new net N$26: U$1.RST, X3-3.KL
- net N$5: now also U$1.D7/GPIO13/RXD2/HSPID/SDA; no longer U$1.D7/GPIO13/RXD2/HSPID
- net N$6: now also U$1.D6/GPIO12/HSPIQ/SCL; no longer U$1.D6/GPIO12/HSPIQ
Changed lines of the file:
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@@
 <?xml version="1.0" encoding="utf-8"?>
 <!DOCTYPE eagle SYSTEM "eagle.dtd">
-<eagle version="7.3.0">
+<eagle version="7.4.0">
 <drawing>
 <settings>
@@
 <part name="X4" library="con-wago-500" deviceset="W237-6" device=""/>
 <part name="J1" library="SparkFun" deviceset="POWER_JACK" device="SMD"/>
+<part name="GND1" library="SparkFun" deviceset="GND" device=""/>
 </parts>
 <sheets>
@@
 <instance part="X4" gate="-6" x="-7.62" y="53.34"/>
 <instance part="J1" gate="G$1" x="17.78" y="5.08"/>
+<instance part="GND1" gate="1" x="50.8" y="15.24"/>
 </instances>
 <busses>
@@
 <segment>
 <pinref part="X2" gate="-1" pin="KL"/>
-<pinref part="U$1" gate="G$1" pin="D6/GPIO12/HSPIQ"/>
+<pinref part="U$1" gate="G$1" pin="D6/GPIO12/HSPIQ/SCL"/>
 <wire x1="116.84" y1="45.72" x2="88.9" y2="45.72" width="0.1524" layer="91"/>
 </segment>
@@
 <wire x1="116.84" y1="40.64" x2="104.14" y2="40.64" width="0.1524" layer="91"/>
 <wire x1="104.14" y1="40.64" x2="104.14" y2="43.18" width="0.1524" layer="91"/>
-<pinref part="U$1" gate="G$1" pin="D7/GPIO13/RXD2/HSPID"/>
+<pinref part="U$1" gate="G$1" pin="D7/GPIO13/RXD2/HSPID/SDA"/>
 <wire x1="104.14" y1="43.18" x2="88.9" y2="43.18" width="0.1524" layer="91"/>
 </segment>
@@
 </segment>
 </net>
-<net name="N$22" class="0">
+<net name="N$23" class="0">
+<segment>
+<pinref part="U$1" gate="G$1" pin="3V3$11"/>
+<wire x1="25.4" y1="40.64" x2="15.24" y2="40.64" width="0.1524" layer="91"/>
+<wire x1="15.24" y1="40.64" x2="15.24" y2="30.48" width="0.1524" layer="91"/>
+<pinref part="X3" gate="-4" pin="KL"/>
+<wire x1="15.24" y1="30.48" x2="-2.54" y2="30.48" width="0.1524" layer="91"/>
+</segment>
+</net>
+<net name="N$26" class="0">
+<segment>
+<pinref part="X3" gate="-3" pin="KL"/>
+<pinref part="U$1" gate="G$1" pin="RST"/>
+<wire x1="-2.54" y1="35.56" x2="25.4" y2="35.56" width="0.1524" layer="91"/>
+</segment>
+</net>
+<net name="GND" class="0">
 <segment>
 <pinref part="U$1" gate="G$1" pin="GND$14"/>
@@
 <pinref part="J1" gate="G$1" pin="PWR"/>
 <wire x1="20.32" y1="12.7" x2="22.86" y2="12.7" width="0.1524" layer="91"/>
-<wire x1="22.86" y1="12.7" x2="22.86" y2="33.02" width="0.1524" layer="91"/>
+<wire x1="22.86" y1="12.7" x2="22.86" y2="22.86" width="0.1524" layer="91"/>
 <junction x="22.86" y="33.02"/>
-</segment>
-</net>
-<net name="N$23" class="0">
-<segment>
-<pinref part="U$1" gate="G$1" pin="3V3$11"/>
-<wire x1="25.4" y1="40.64" x2="15.24" y2="40.64" width="0.1524" layer="91"/>
-<wire x1="15.24" y1="40.64" x2="15.24" y2="30.48" width="0.1524" layer="91"/>
-<pinref part="X3" gate="-4" pin="KL"/>
-<wire x1="15.24" y1="30.48" x2="-2.54" y2="30.48" width="0.1524" layer="91"/>
-</segment>
-</net>
+<pinref part="U$1" gate="G$1" pin="GND$10"/>
+<wire x1="22.86" y1="22.86" x2="22.86" y2="33.02" width="0.1524" layer="91"/>
+<wire x1="25.4" y1="43.18" x2="22.86" y2="43.18" width="0.1524" layer="91"/>
+<wire x1="22.86" y1="43.18" x2="22.86" y2="33.02" width="0.1524" layer="91"/>
+<pinref part="U$1" gate="G$1" pin="GND$24"/>
+<wire x1="88.9" y1="50.8" x2="91.44" y2="50.8" width="0.1524" layer="91"/>
+<wire x1="91.44" y1="50.8" x2="91.44" y2="33.02" width="0.1524" layer="91"/>
+<wire x1="91.44" y1="33.02" x2="91.44" y2="22.86" width="0.1524" layer="91"/>
+<wire x1="91.44" y1="22.86" x2="50.8" y2="22.86" width="0.1524" layer="91"/>
+<junction x="22.86" y="22.86"/>
+<pinref part="U$1" gate="G$1" pin="GND$17"/>
+<wire x1="50.8" y1="22.86" x2="22.86" y2="22.86" width="0.1524" layer="91"/>
+<wire x1="88.9" y1="33.02" x2="91.44" y2="33.02" width="0.1524" layer="91"/>
+<junction x="91.44" y="33.02"/>
+<pinref part="GND1" gate="1" pin="GND"/>
+<wire x1="50.8" y1="17.78" x2="50.8" y2="22.86" width="0.1524" layer="91"/>
+<junction x="50.8" y="22.86"/>
+</segment>
+</net>

Commit message: Updated the i2c pins to all shields to use d11/d12  as these pins will have dual use with the upcoming wifimcu Added FM24W256  Fram shield Added X95840 Digital potentiometer Shield Added AD5696 DAC Shield
Connections:
- net GND: no longer U$1.GND$24
Changed lines of the file:
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@@
 <wire x1="25.4" y1="43.18" x2="22.86" y2="43.18" width="0.1524" layer="91"/>
 <wire x1="22.86" y1="43.18" x2="22.86" y2="33.02" width="0.1524" layer="91"/>
-<pinref part="U$1" gate="G$1" pin="GND$24"/>
-<wire x1="88.9" y1="50.8" x2="91.44" y2="50.8" width="0.1524" layer="91"/>
-<wire x1="91.44" y1="50.8" x2="91.44" y2="33.02" width="0.1524" layer="91"/>
 <wire x1="91.44" y1="33.02" x2="91.44" y2="22.86" width="0.1524" layer="91"/>
 <wire x1="91.44" y1="22.86" x2="50.8" y2="22.86" width="0.1524" layer="91"/>
@@
 <wire x1="50.8" y1="22.86" x2="22.86" y2="22.86" width="0.1524" layer="91"/>
 <wire x1="88.9" y1="33.02" x2="91.44" y2="33.02" width="0.1524" layer="91"/>
-<junction x="91.44" y="33.02"/>
 <pinref part="GND1" gate="1" pin="GND"/>
 <wire x1="50.8" y1="17.78" x2="50.8" y2="22.86" width="0.1524" layer="91"/>
