File: LIS331_Accelerometer/LIS331_Accelerometer.sch (EAGLE design)
At the start: 8 parts, among them U1 LIS331

Commit message: Added OLED Shield Added LiPo Battery Charger Shield Updated outlines of all shields to match the cutout of the nodemcu board
Parts:
- removed JP1: JP1, SparkFun:M03PTH
- added SJ1: (no value), SparkFun:SOLDERJUMPER_2WAYT
Connections:
- net +3V3: now also SJ1.1; no longer JP1.1
- net GND: now also SJ1.3; no longer JP1.3, U$2.MO/MOSI/SDCMD
- net N$6: now also SJ1.2; no longer JP1.2
Changed lines of the file:
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@@
 <?xml version="1.0" encoding="utf-8"?>
 <!DOCTYPE eagle SYSTEM "eagle.dtd">
-<eagle version="7.3.0">
+<eagle version="7.4.0">
 <drawing>
 <settings>
@@
 <parts>
 <part name="GND1" library="SparkFun" deviceset="GND" device=""/>
-<part name="GND2" library="SparkFun" deviceset="GND" device=""/>
 <part name="GND4" library="SparkFun" deviceset="GND" device=""/>
 <part name="C1" library="SparkFun" deviceset="CAP" device="0603-CAP" value=".1uF"/>
@@
 <part name="C3" library="SparkFun" deviceset="CAP_POL" device="1206" value="10uF"/>
 <part name="GND3" library="SparkFun" deviceset="GND" device=""/>
-<part name="JP1" library="SparkFun" deviceset="M03" device="PTH" value="JP1"/>
 <part name="GND7" library="SparkFun" deviceset="GND" device=""/>
 <part name="JP2" library="SparkFun" deviceset="M02" device="PTH" value="JP2"/>
@@
 <part name="GND5" library="SparkFun" deviceset="GND" device=""/>
 <part name="GND6" library="SparkFun" deviceset="GND" device=""/>
+<part name="SJ1" library="SparkFun" deviceset="SOLDERJUMPER_2WAY" device="T"/>
 </parts>
 <sheets>
@@
 <instances>
 <instance part="GND1" gate="1" x="93.98" y="55.88"/>
-<instance part="GND2" gate="1" x="10.16" y="53.34"/>
 <instance part="GND4" gate="1" x="88.9" y="81.28"/>
 <instance part="C1" gate="G$1" x="88.9" y="88.9"/>
@@
 <instance part="C3" gate="G$1" x="76.2" y="91.44"/>
 <instance part="GND3" gate="1" x="76.2" y="81.28"/>
-<instance part="JP1" gate="G$1" x="172.72" y="63.5" rot="R180"/>
-<instance part="GND7" gate="1" x="160.02" y="55.88"/>
+<instance part="GND7" gate="1" x="167.64" y="38.1"/>
 <instance part="JP2" gate="G$1" x="152.4" y="66.04" rot="R180"/>
 <instance part="U$2" gate="G$1" x="27.94" y="53.34"/>
@@
 <instance part="GND5" gate="1" x="2.54" y="27.94"/>
 <instance part="GND6" gate="1" x="76.2" y="25.4"/>
+<instance part="SJ1" gate="G$1" x="167.64" y="63.5"/>
 </instances>
 <busses>
@@
 </segment>
 <segment>
-<wire x1="165.1" y1="60.96" x2="160.02" y2="60.96" width="0.1524" layer="91"/>
-<wire x1="160.02" y1="60.96" x2="160.02" y2="58.42" width="0.1524" layer="91"/>
-<pinref part="JP1" gate="G$1" pin="3"/>
+<wire x1="167.64" y1="58.42" x2="167.64" y2="40.64" width="0.1524" layer="91"/>
 <pinref part="GND7" gate="1" pin="GND"/>
-</segment>
-<segment>
-<pinref part="GND2" gate="1" pin="GND"/>
-<pinref part="U$2" gate="G$1" pin="MO/MOSI/SDCMD"/>
+<pinref part="SJ1" gate="G$1" pin="3"/>
 </segment>
 <segment>
@@
 <wire x1="96.52" y1="78.74" x2="96.52" y2="96.52" width="0.1524" layer="91"/>
 <wire x1="96.52" y1="96.52" x2="142.24" y2="96.52" width="0.1524" layer="91"/>
-<wire x1="142.24" y1="96.52" x2="162.56" y2="96.52" width="0.1524" layer="91"/>
-<wire x1="162.56" y1="96.52" x2="172.72" y2="96.52" width="0.1524" layer="91"/>
+<wire x1="142.24" y1="96.52" x2="167.64" y2="96.52" width="0.1524" layer="91"/>
+<wire x1="167.64" y1="96.52" x2="172.72" y2="96.52" width="0.1524" layer="91"/>
 <wire x1="172.72" y1="93.98" x2="172.72" y2="96.52" width="0.1524" layer="91"/>
 <wire x1="172.72" y1="96.52" x2="177.8" y2="96.52" width="0.1524" layer="91"/>
@@
 <wire x1="139.7" y1="78.74" x2="142.24" y2="78.74" width="0.1524" layer="91"/>
 <wire x1="142.24" y1="78.74" x2="142.24" y2="96.52" width="0.1524" layer="91"/>
-<wire x1="165.1" y1="66.04" x2="162.56" y2="66.04" width="0.1524" layer="91"/>
-<wire x1="162.56" y1="66.04" x2="162.56" y2="96.52" width="0.1524" layer="91"/>
+<wire x1="167.64" y1="68.58" x2="167.64" y2="96.52" width="0.1524" layer="91"/>
 <junction x="88.9" y="96.52"/>
 <junction x="96.52" y="76.2"/>
@@
 <junction x="172.72" y="96.52"/>
 <junction x="142.24" y="96.52"/>
-<junction x="162.56" y="96.52"/>
+<junction x="167.64" y="96.52"/>
 <pinref part="C1" gate="G$1" pin="1"/>
 <pinref part="+3V2" gate="G$1" pin="+3V3"/>
@@
 <pinref part="C3" gate="G$1" pin="+"/>
 <pinref part="U1" gate="G$1" pin="CS"/>
-<pinref part="JP1" gate="G$1" pin="1"/>
+<pinref part="SJ1" gate="G$1" pin="1"/>
 </segment>
 <segment>
@@
 <net name="N$6" class="0">
 <segment>
-<wire x1="165.1" y1="63.5" x2="160.02" y2="63.5" width="0.1524" layer="91"/>
+<wire x1="162.56" y1="63.5" x2="160.02" y2="63.5" width="0.1524" layer="91"/>
 <wire x1="160.02" y1="63.5" x2="160.02" y2="71.12" width="0.1524" layer="91"/>
 <wire x1="160.02" y1="71.12" x2="139.7" y2="71.12" width="0.1524" layer="91"/>
-<pinref part="JP1" gate="G$1" pin="2"/>
 <pinref part="U1" gate="G$1" pin="SA0/SDO"/>
-</segment>
-</net>
+<pinref part="SJ1" gate="G$1" pin="2"/>
+</segment>
+</net>

Commit message: Updated the i2c pins to all shields to use d11/d12  as these pins will have dual use with the upcoming wifimcu Added FM24W256  Fram shield Added X95840 Digital potentiometer Shield Added AD5696 DAC Shield
Connections:
- net GND: no longer U$2.GND$24
- net N$2: now also U$2.D11/GPIO09/SDD2; no longer U$2.D7/GPIO13/RXD2/HSPID/SDA
- net N$5: now also U$2.D12/GPIO10/SDD3; no longer U$2.D6/GPIO12/HSPIQ/SCL
Changed lines of the file:
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@@
 <pinref part="GND6" gate="1" pin="GND"/>
 <wire x1="76.2" y1="27.94" x2="76.2" y2="38.1" width="0.1524" layer="91"/>
-<pinref part="U$2" gate="G$1" pin="GND$24"/>
-<wire x1="76.2" y1="38.1" x2="76.2" y2="55.88" width="0.1524" layer="91"/>
-<wire x1="76.2" y1="55.88" x2="73.66" y2="55.88" width="0.1524" layer="91"/>
 <pinref part="U$2" gate="G$1" pin="GND$17"/>
 <wire x1="73.66" y1="38.1" x2="76.2" y2="38.1" width="0.1524" layer="91"/>
-<junction x="76.2" y="38.1"/>
 </segment>
 <segment>
@@
 <pinref part="R1" gate="G$1" pin="1"/>
 <pinref part="U1" gate="G$1" pin="SDA/SDI"/>
-<wire x1="218.44" y1="73.66" x2="218.44" y2="48.26" width="0.1524" layer="91"/>
-<wire x1="218.44" y1="48.26" x2="73.66" y2="48.26" width="0.1524" layer="91"/>
-<pinref part="U$2" gate="G$1" pin="D7/GPIO13/RXD2/HSPID/SDA"/>
-<wire x1="175.26" y1="73.66" x2="218.44" y2="73.66" width="0.1524" layer="91"/>
+<wire x1="175.26" y1="73.66" x2="190.5" y2="73.66" width="0.1524" layer="91"/>
+<wire x1="190.5" y1="73.66" x2="190.5" y2="116.84" width="0.1524" layer="91"/>
+<wire x1="190.5" y1="116.84" x2="0" y2="116.84" width="0.1524" layer="91"/>
+<wire x1="0" y1="116.84" x2="0" y2="60.96" width="0.1524" layer="91"/>
+<pinref part="U$2" gate="G$1" pin="D11/GPIO09/SDD2"/>
+<wire x1="0" y1="60.96" x2="10.16" y2="60.96" width="0.1524" layer="91"/>
 </segment>
 </net>
@@
 <pinref part="R2" gate="G$1" pin="1"/>
 <pinref part="U1" gate="G$1" pin="SCL/SPC"/>
-<wire x1="73.66" y1="50.8" x2="220.98" y2="50.8" width="0.1524" layer="91"/>
-<wire x1="220.98" y1="50.8" x2="220.98" y2="76.2" width="0.1524" layer="91"/>
-<wire x1="177.8" y1="76.2" x2="220.98" y2="76.2" width="0.1524" layer="91"/>
-<pinref part="U$2" gate="G$1" pin="D6/GPIO12/HSPIQ/SCL"/>
+<wire x1="177.8" y1="76.2" x2="185.42" y2="76.2" width="0.1524" layer="91"/>
+<wire x1="185.42" y1="76.2" x2="185.42" y2="111.76" width="0.1524" layer="91"/>
+<wire x1="185.42" y1="111.76" x2="2.54" y2="111.76" width="0.1524" layer="91"/>
+<wire x1="2.54" y1="111.76" x2="2.54" y2="63.5" width="0.1524" layer="91"/>
+<pinref part="U$2" gate="G$1" pin="D12/GPIO10/SDD3"/>
+<wire x1="2.54" y1="63.5" x2="10.16" y2="63.5" width="0.1524" layer="91"/>
 </segment>
 </net>
