File: OLED_Shield/OLED_Shield.brd (EAGLE design)
At the start: 84.6 x 35.2 mm, 8 parts

Commit message: Updated the i2c pins to all shields to use d11/d12  as these pins will have dual use with the upcoming wifimcu Added FM24W256  Fram shield Added X95840 Digital potentiometer Shield Added AD5696 DAC Shield
Parts:
- moved R1 20.4 mm to (46.5, 20.0), turned to 180 degrees
- moved R2 17.3 mm to (46.5, 22.5), turned to 180 degrees
Connections:
- net GND: no longer U$1.24
- net N$2: now also U$1.5; no longer U$1.21
- net N$3: now also U$1.4; no longer U$1.22
Routing:
- net N$2: track 99.4 -> 120.4 mm, vias 3 -> 4
- net N$3: track 108.7 -> 117.1 mm
- net 3.3V: track 93.6 -> 97.9 mm
Changed lines of the file:
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@@
 <elements>
 <element name="C1" library="SparkFun" package="0402-CAP" value="0.1uF" x="42.43" y="25.43" rot="R270"/>
-<element name="R1" library="SparkFun" package="0402-RES" value="4.7k" x="27.12" y="26.19" rot="R270"/>
-<element name="R2" library="SparkFun" package="0402-RES" value="4.7k" x="29.66" y="26.19" rot="R270"/>
+<element name="R1" library="SparkFun" package="0402-RES" value="4.7k" x="46.53" y="19.98" rot="R180"/>
+<element name="R2" library="SparkFun" package="0402-RES" value="4.7k" x="46.52" y="22.52" rot="R180"/>
 <element name="U$1" library="NerduinoShieldLib" package="NERDUINO_STACK" value="NERDSHIELD" x="24.58" y="12.22"/>
 <element name="JP1" library="SparkFun" package="1X04_NO_SILK" value="" x="51.43" y="14.89" rot="R90"/>
@@
 <contactref element="C1" pad="2"/>
 <contactref element="U$1" pad="10"/>
-<contactref element="U$1" pad="24"/>
 <contactref element="U$1" pad="17"/>
 <contactref element="JP1" pad="2"/>
@@
 <wire x1="42.36" y1="30" x2="42.36" y2="28.11" width="0.254" layer="1"/>
 <wire x1="42.36" y1="28.11" x2="42.43" y2="26.08" width="0.254" layer="1"/>
-<wire x1="27.12" y1="25.54" x2="29.66" y2="25.54" width="0.254" layer="1"/>
 <contactref element="JP4" pad="1"/>
 <contactref element="JP3" pad="1"/>
 <contactref element="JP1" pad="1"/>
 <contactref element="JP2" pad="1"/>
-<wire x1="42.43" y1="26.08" x2="52" y2="26.08" width="0.254" layer="1"/>
+<wire x1="42.43" y1="26.08" x2="44.11" y2="26.08" width="0.254" layer="1"/>
+<wire x1="44.11" y1="26.08" x2="52" y2="26.08" width="0.254" layer="1"/>
 <wire x1="52" y1="26.08" x2="60.31" y2="34.39" width="0.254" layer="1"/>
 <wire x1="60.31" y1="34.39" x2="62.64" y2="34.39" width="0.254" layer="1"/>
@@
 <wire x1="59.56" y1="16.86" x2="55.11" y2="16.86" width="0.254" layer="1"/>
 <wire x1="55.11" y1="16.86" x2="55.03" y2="16.94" width="0.254" layer="1"/>
-<wire x1="29.66" y1="25.54" x2="42.43" y2="26.08" width="0" layer="19" extent="1-1"/>
+<wire x1="45.88" y1="19.98" x2="45.88" y2="22.51" width="0.254" layer="1"/>
+<wire x1="45.88" y1="22.51" x2="45.87" y2="22.52" width="0.254" layer="1"/>
+<wire x1="45.87" y1="22.52" x2="45.87" y2="24.32" width="0.254" layer="1"/>
+<wire x1="45.87" y1="24.32" x2="44.11" y2="26.08" width="0.254" layer="1"/>
 </signal>
 <signal name="N$2">
 <contactref element="R2" pad="1"/>
-<contactref element="U$1" pad="21"/>
-<wire x1="29.66" y1="30" x2="29.66" y2="26.84" width="0.254" layer="1"/>
 <contactref element="JP1" pad="4"/>
 <contactref element="JP2" pad="4"/>
 <contactref element="JP3" pad="4"/>
 <contactref element="JP4" pad="4"/>
-<wire x1="29.66" y1="26.84" x2="37.39" y2="26.84" width="0.254" layer="1"/>
-<wire x1="37.39" y1="26.84" x2="41.7" y2="22.53" width="0.254" layer="1"/>
-<wire x1="41.7" y1="22.53" x2="51.41" y2="22.53" width="0.254" layer="1"/>
-<wire x1="51.41" y1="22.53" x2="51.43" y2="22.51" width="0.254" layer="1"/>
-<wire x1="51.43" y1="22.51" x2="61.09" y2="22.51" width="0.254" layer="16"/>
+<wire x1="51.43" y1="22.51" x2="61.33" y2="22.51" width="0.254" layer="16"/>
 <wire x1="61.33" y1="22.51" x2="61.64" y2="22.51" width="0.254" layer="16"/>
 <wire x1="61.64" y1="22.51" x2="70.58" y2="31.45" width="0.254" layer="16"/>
@@
 <wire x1="63.48" y1="20.36" x2="61.33" y2="22.51" width="0.254" layer="1"/>
 <via x="61.33" y="22.51" extent="1-16" drill="0.5"/>
-<wire x1="61.33" y1="22.51" x2="61.09" y2="22.51" width="0.254" layer="16"/>
+<contactref element="U$1" pad="5"/>
+<wire x1="47.17" y1="22.52" x2="51.42" y2="22.52" width="0.254" layer="1"/>
+<wire x1="51.42" y1="22.52" x2="51.43" y2="22.51" width="0.254" layer="1"/>
+<wire x1="16.96" y1="7.14" x2="16.96" y2="9.08" width="0.254" layer="1"/>
+<wire x1="16.96" y1="9.08" x2="18.52" y2="10.64" width="0.254" layer="1"/>
+<wire x1="18.52" y1="10.64" x2="42.17" y2="10.64" width="0.254" layer="1"/>
+<wire x1="42.17" y1="10.64" x2="47.3" y2="15.77" width="0.254" layer="1"/>
+<via x="47.3" y="15.77" extent="1-16" drill="0.5"/>
+<wire x1="47.3" y1="15.77" x2="47.3" y2="18.38" width="0.254" layer="16"/>
+<wire x1="47.3" y1="18.38" x2="51.43" y2="22.51" width="0.254" layer="16"/>
 </signal>
 <signal name="N$3">
 <contactref element="R1" pad="1"/>
-<contactref element="U$1" pad="22"/>
-<wire x1="27.12" y1="30" x2="27.12" y2="26.84" width="0.254" layer="1"/>
 <contactref element="JP1" pad="3"/>
 <contactref element="JP2" pad="3"/>
 <contactref element="JP3" pad="3"/>
 <contactref element="JP4" pad="3"/>
-<wire x1="27.12" y1="26.84" x2="26.35" y2="26.84" width="0.254" layer="1"/>
-<wire x1="26.35" y1="26.84" x2="25.06" y2="25.55" width="0.254" layer="1"/>
-<wire x1="25.06" y1="25.55" x2="25.06" y2="22.22" width="0.254" layer="1"/>
-<wire x1="25.06" y1="22.22" x2="27.32" y2="19.96" width="0.254" layer="1"/>
-<wire x1="27.32" y1="19.96" x2="51.42" y2="19.96" width="0.254" layer="1"/>
-<wire x1="51.42" y1="19.96" x2="51.43" y2="19.97" width="0.254" layer="1"/>
 <wire x1="51.43" y1="19.97" x2="61.56" y2="19.97" width="0.254" layer="16"/>
 <wire x1="61.56" y1="19.97" x2="70.81" y2="29.22" width="0.254" layer="16"/>
@@
 <wire x1="66.06" y1="17.68" x2="66.06" y2="21.85" width="0.254" layer="1"/>
 <wire x1="66.06" y1="21.85" x2="64.75" y2="23.16" width="0.254" layer="1"/>
+<contactref element="U$1" pad="4"/>
+<wire x1="47.18" y1="19.98" x2="51.42" y2="19.98" width="0.254" layer="1"/>
+<wire x1="51.42" y1="19.98" x2="51.43" y2="19.97" width="0.254" layer="1"/>
+<wire x1="14.42" y1="7.14" x2="14.42" y2="9.31" width="0.254" layer="1"/>
+<wire x1="14.42" y1="9.31" x2="17.44" y2="12.33" width="0.254" layer="1"/>
+<wire x1="17.44" y1="12.33" x2="41.15" y2="12.33" width="0.254" layer="1"/>
+<wire x1="41.15" y1="12.33" x2="47.37" y2="18.55" width="0.254" layer="1"/>
+<wire x1="47.37" y1="18.55" x2="47.37" y2="19.79" width="0.254" layer="1"/>
+<wire x1="47.37" y1="19.79" x2="47.18" y2="19.98" width="0.254" layer="1"/>
 <wire x1="61.56" y1="19.97" x2="64.75" y2="23.16" width="0" layer="19" extent="1-16"/>
 </signal>
