File: PIR_Shield/PIR_Shield.sch (EAGLE design)
At the start: 13 parts

Commit message: Updated the i2c pins to all shields to use d11/d12  as these pins will have dual use with the upcoming wifimcu Added FM24W256  Fram shield Added X95840 Digital potentiometer Shield Added AD5696 DAC Shield
Connections:
- net GND: no longer U$1.GND$24
Changed lines of the file:
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@@
 </segment>
 <segment>
-<pinref part="U$1" gate="G$1" pin="GND$24"/>
 <pinref part="GND4" gate="1" pin="GND"/>
-<wire x1="71.12" y1="50.8" x2="76.2" y2="50.8" width="0.1524" layer="91"/>
-<wire x1="76.2" y1="50.8" x2="76.2" y2="33.02" width="0.1524" layer="91"/>
 <pinref part="U$1" gate="G$1" pin="GND$17"/>
 <wire x1="76.2" y1="33.02" x2="76.2" y2="20.32" width="0.1524" layer="91"/>
 <wire x1="71.12" y1="33.02" x2="76.2" y2="33.02" width="0.1524" layer="91"/>
-<junction x="76.2" y="33.02"/>
 </segment>
 <segment>
